File: lm2596 current limited charger.brd (EAGLE design)
At the start: 160 x 100 mm, 53 parts, among them IC1 TLC339D, IC2 MCP602SN, IC5 LD117AS33TR

Commit message: upd
Parts:
- removed C11, C13: (no value), rcl:PANASONIC_C
- removed R20: VOLTS, pot:B64Y
- added C48: 10uF 50V, SparkFun:EIA3216
- added C5: (no value), resistor:E3,5-8
- added C56: 220µF 50V, rcl:E3,5-10
- added C6, C7: 10uF, rcl:C1206K
- added D13, D18: SS34, dp_devices:DO-214AC
- added IC9: XL1509-5.0E1, Cohesion_parts:SO08
- added L2: 68uH, rc-master-smd:CD75
- added R24: VOLTS, pot:B64Y
- added TP1, TP2: TPPAD1-20Y, testpad:P1-20Y
- D1: value 250mA/100V -> 1N4148
- moved C4 334.8 mm to (46.4, 61.4), turned to 180 degrees
- moved R63 322.8 mm to (8.40, 66.4), turned to 180 degrees
- moved R62 318.3 mm to (8.40, 63.4), turned to 180 degrees
- moved R23 314.8 mm to (51.4, 32.4)
- moved U$24 314.5 mm to (8.40, 74.4)
- moved C3 298.5 mm to (54.3, 58.9), turned to 180 degrees
- moved D11 295.1 mm to (53.2, 87.4), turned to 90 degrees
- moved IC5 288.9 mm to (53.2, 68.4), turned to 180 degrees
- moved D12 287.9 mm to (8.40, 58.4)
- moved R22 285.7 mm to (53.2, 81.4), turned to 270 degrees
- moved BATT 281.5 mm to (33.1, 4.60), turned to 180 degrees
- moved R21 263.0 mm to (46.4, 64.4), turned to 180 degrees
- moved D10 247.3 mm to (58.2, 87.4), turned to 90 degrees
- moved R15 236.7 mm to (49.4, 43.4), turned to 270 degrees
- moved R13 233.6 mm to (58.2, 81.4), turned to 270 degrees
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Connections:
- removed net 3.3V: C13.+, IC5.4, R18.E
- new net 5VREG: C56.+, IC9.3, L2.1
- new net N$25: D18.1, IC9.2, L2.2
- new net N$26: D13.1, IC9.1
- net 13V8: now also R24.E; no longer R20.A
- net 3V3: now also C7.1, IC5.4, R18.E
- net BATT+: now also C48.A, C5.+, D13.2, TP1.TP
- net BATT-: now also TP2.TP; no longer R63.1, U$24.3
- net FEEDBACK: now also R24.A, R24.S; no longer R20.E, R20.S
- net GND: now also C6.2, C7.2, R63.1, U$24.3; no longer C11.-, C13.-
- net OUT-: now also C48.C, C5.-, C56.-, D18.2, IC9.4, IC9.5, IC9.6, IC9.7, IC9.8
- net SOLAR-IN+: now also C6.1; no longer C11.+
Routing:
- net BATT-: track 0.00 -> 91.8 mm
- net 13V8: track 0.00 -> 84.5 mm
- net BATT+: track 0.00 -> 79.0 mm
- net FEEDBACK: track 0.00 -> 60.3 mm
- net N$19: track 0.00 -> 53.3 mm
- net 3V3: track 0.00 -> 42.0 mm
- net N$18: track 0.00 -> 41.7 mm
- net SOLAR-IN+: track 0.00 -> 40.8 mm
- net N$7: track 0.00 -> 37.8 mm
- net N$17: track 0.00 -> 30.0 mm
- net GND: track 0.00 -> 24.7 mm, vias 0 -> 41
- net N$6: track 0.00 -> 18.8 mm
- net N$21: track 0.00 -> 12.7 mm
- net N$5: track 0.00 -> 12.3 mm
- net N$3: track 0.00 -> 11.8 mm
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- added copper zone on layer 1, net 13V8
- added copper zone on layer 1, net BATT+
- added copper zone on layer 1, net BATT-
- added copper zone on layer 1, net GND
- added copper zone on layer 1, net N$1
- added copper zone on layer 1, net OUT-
- added copper zone on layer 1, net SOLAR-IN+
Other:
- board size 160 x 100 mm -> 65 x 151 mm
- board text added: "+"
- board text added: "-"
- board text added: "todo USB Charge LED FAN"

Commit message: as ordered
Parts:
- removed BATT: (no value), con-wago-500:W237-102
- removed C48: 10uF 50V, SparkFun:EIA3216
- removed C5: (no value), resistor:E3,5-8
- removed C56: 220µF 50V, rcl:E3,5-10
- removed D13, D18: SS34, dp_devices:DO-214AC
- removed IC9: XL1509-5.0E1, Cohesion_parts:SO08
- removed L2: 68uH, rc-master-smd:CD75
- added U$2, U$3: PCB-6.35MM-RA-SPADE, AUTOMOTIVERELAYS:PCB-6.35MM-RA-SPADE
- D10: value LIMIT -> FLOAT
- moved D8 4.12 mm to (25.8, 39.2)
- moved R19 3.00 mm to (48.4, 37.4)
- moved R23 3.00 mm to (48.4, 32.4)
- moved C2 2.50 mm to (35.1, 35.6)
- moved TP1 0.50 mm to (5.50, 35.0), turned to 180 degrees
- moved TP2 0.50 mm to (59.5, 35.0), turned to 180 degrees
- moved C4 0.30 mm to (46.4, 61.1)
- moved R15 0.20 mm to (49.2, 43.4)
- moved R21 0.20 mm to (46.4, 64.6)
- renumbered SOLAR to CHARGERIN
Connections:
- removed net 5VREG: C56.+, IC9.3, L2.1
- removed net N$25: D18.1, IC9.2, L2.2
- removed net N$26: D13.1, IC9.1
- net BATT+: now also U$2.P$1, U$2.P$2; no longer BATT.2, C48.A, C5.+, D13.2
- net BATT-: now also U$3.P$1, U$3.P$2; no longer BATT.1
- net OUT-: no longer C48.C, C5.-, C56.-, D18.2, IC9.4, IC9.5, IC9.6, IC9.7, IC9.8
Routing:
- net GND: track 24.7 -> 23.1 mm, vias 41 -> 82
- added copper zone on layer 16, net GND
Other:
- board size 65 x 151 mm -> 65 x 68 mm
- board text added: "BATT+"
- board text added: "BATT-"
- board text removed: "todo USB Charge LED FAN"
