File: lm2596 current limited charger.sch (EAGLE design)
At the start: 53 parts, among them IC1 TLC339D, IC2 MCP602SN, IC5 LD117AS33TR

Commit message: upd
Parts:
- removed C11, C13: (no value), rcl:CPOL-EUC
- removed R20: VOLTS, pot:TRIM_EU-B64Y
- added C48: 10uF 50V, SparkFun:CAP_POL1206
- added C5: (no value), resistor:CPOL-EUE3.5-8
- added C56: 220µF 50V, rcl:CPOL-EUE3.5-10
- added C6, C7: 10uF, rcl:C-EUC1206K
- added D13, D18: SS34, dp_devices:DIODE-DO-214AC
- added IC9: XL1509-5.0E1, Cohesion_parts:XL1509
- added L2: 68uH, rc-master-smd:L_CD75
- added R24: VOLTS, pot:TRIM_EU-B64Y
- added TP1, TP2: TPPAD1-20Y, testpad:TPPAD1-20Y
- D1: value 250mA/100V -> 1N4148
Connections:
- removed net 3.3V: C13.+, IC5.OUT, R18.E
- new net 5VREG: C56.+, IC9.FB, L2.1
- new net N$25: D18.C, IC9.OUT, L2.2
- new net N$26: D13.C, IC9.IN
- net 13V8: now also R24.E; no longer R20.A
- net 3V3: now also C7.1, IC5.OUT, R18.E
- net BATT+: now also C48.+, C5.+, D13.A, TP1.TP
- net BATT-: now also TP2.TP; no longer R63.1, U$24.S
- net FEEDBACK: now also R24.A, R24.S; no longer R20.E, R20.S
- net GND: now also C6.2, C7.2, R63.1, U$24.S; no longer C11.-, C13.-
- net OUT-: now also C48.-, C5.-, C56.-, D18.A, IC9.EN, IC9.GND1, IC9.GND2, IC9.GND3, IC9.GND4
- net SOLAR-IN+: now also C6.1; no longer C11.+

Commit message: as ordered
Parts:
- removed BATT: (no value), con-wago-500:W237-102
- removed C48: 10uF 50V, SparkFun:CAP_POL1206
- removed C5: (no value), resistor:CPOL-EUE3.5-8
- removed C56: 220µF 50V, rcl:CPOL-EUE3.5-10
- removed D13, D18: SS34, dp_devices:DIODE-DO-214AC
- removed IC9: XL1509-5.0E1, Cohesion_parts:XL1509
- removed L2: 68uH, rc-master-smd:L_CD75
- added U$2, U$3: PCB-6.35MM-RA-SPADE, AUTOMOTIVERELAYS:PCB-6.35MM-RA-SPADE
- D10: value LIMIT -> FLOAT
- renumbered SOLAR to CHARGERIN
Connections:
- removed net 5VREG: C56.+, IC9.FB, L2.1
- removed net N$25: D18.C, IC9.OUT, L2.2
- removed net N$26: D13.C, IC9.IN
- net BATT+: now also U$2.P$1; no longer BATT-2.KL, C48.+, C5.+, D13.A
- net BATT-: now also U$3.P$1; no longer BATT-1.KL
- net OUT-: no longer C48.-, C5.-, C56.-, D18.A, IC9.EN, IC9.GND1, IC9.GND2, IC9.GND3, IC9.GND4
